Commit message: Your descriptive commit message here

File: greenguard_description/urdf/greenguard.urdf.xacro (robot description, xacro)
@@ -70,9 +70,31 @@
         </xacro:inertial_box>
     </link>
+    <!-- IMU Sensor Definations -->
+    <link name="imu_link">
+        <visual>
+            <geometry>
+            <box size="0.1 0.1 0.1"/>
+            </geometry>
+        </visual>
+        <collision>
+            <geometry>
+            <box size="0.1 0.1 0.1"/>
+            </geometry>
+        </collision>
+        <xacro:inertial_box mass="0.1" x="0.12" y="0.15" z="0.15">
+            <origin xyz="0.0 0 0" rpy="0 0 0"/>
+        </xacro:inertial_box>
+    </link>
+    <joint name="imu_joint" type="fixed">
+        <parent link="base_link"/>
+        <child link="imu_link"/>
+        <origin xyz="0 0 0.01"/>
+    </joint>
+    <!-- End of IMU Sensor Definations -->
     <xacro:wheel name="front_right" x="${base_x/2}" y="${base_y/2}" z="${base_z/3}" wheel_radius="${wheel_radius}" wheel_width="${wheel_width}" velocity="${velocity}" effort="${effort}" mass="${wheel_mass}"/>
     <xacro:wheel name="front_left" x="${base_x/2}" y="-${base_y/2}" z="${base_z/3}" wheel_radius="${wheel_radius}" wheel_width="${wheel_width}" velocity="${velocity}" effort="${effort}" mass="${wheel_mass}"/>
     <xacro:wheel name="rear_right" x="-${base_x/2}" y="${base_y/2}" z="${base_z/3}" wheel_radius="${wheel_radius}" wheel_width="${wheel_width}" velocity="${velocity}" effort="${effort}" mass="${wheel_mass}"/>
     <xacro:wheel name="rear_left" x="-${base_x/2}" y="-${base_y/2}" z="${base_z/3}" wheel_radius="${wheel_radius}" wheel_width="${wheel_width}" velocity="${velocity}" effort="${effort}" mass="${wheel_mass}"/>
-    <!-- camera_joint describes where the camera is relative to the arm -->
+        <!-- - camera_joint describes where the camera is relative to the arm -->
     <!-- - Even though the camera isn't moving relative to the arm, it will probably be helpful to have its own link/frame rather than just adding more visuals to the arm -->
     <!-- - For this example, the camera_link origin will be at the centre of the camera's "sensor" -->
@@ -82,5 +104,5 @@
         <child link="camera_link"/>
     </joint>
-    <!-- camera_link describes the camera at the end of the arm -->
+    <!-- - camera_link describes the camera at the end of the arm -->
     <!-- - It has multiple visual elements, which ultimately get combined together -->
     <!-- - Even if we specify different materials, RViz will just colour them all the same as the first -->

File: greenguard_description/urdf/greenguard_gazebo.xacro (robot description, xacro)
@@ -53,4 +53,72 @@
     <!-- Note that although visualise is set to true, it won't actually visualise the depth camera in gazebo. To see the preview,
             try swapping "depth" to "camera"-->
+    <gazebo reference="imu_link">
+        <sensor name="imu_sensor" type="imu">
+        <plugin filename="libgazebo_ros_imu_sensor.so" name="imu_plugin">
+            <ros>
+                <namespace>/demo</namespace>
+                <remapping>~/out:=imu</remapping>
+            </ros>
+            <initial_orientation_as_reference>false</initial_orientation_as_reference>
+            </plugin>
+            <always_on>true</always_on>
+            <update_rate>100</update_rate>
+            <visualize>true</visualize>
+            <imu>
+            <angular_velocity>
+                <x>
+                <noise type="gaussian">
+                    <mean>0.0</mean>
+                    <stddev>2e-4</stddev>
+                    <bias_mean>0.0000075</bias_mean>
+                    <bias_stddev>0.0000008</bias_stddev>
+                </noise>
+                </x>
+                <y>
+                <noise type="gaussian">
+                    <mean>0.0</mean>
+                    <stddev>2e-4</stddev>
+                    <bias_mean>0.0000075</bias_mean>
+                    <bias_stddev>0.0000008</bias_stddev>
+                </noise>
+                </y>
+                <z>
+                <noise type="gaussian">
+                    <mean>0.0</mean>
+                    <stddev>2e-4</stddev>
+                    <bias_mean>0.0000075</bias_mean>
+                    <bias_stddev>0.0000008</bias_stddev>
+                </noise>
+                </z>
+            </angular_velocity>
+            <linear_acceleration>
+                <x>
+                <noise type="gaussian">
+                    <mean>0.0</mean>
+                    <stddev>1.7e-2</stddev>
+                    <bias_mean>0.1</bias_mean>
+                    <bias_stddev>0.001</bias_stddev>
+                </noise>
+                </x>
+                <y>
+                <noise type="gaussian">
+                    <mean>0.0</mean>
+                    <stddev>1.7e-2</stddev>
+                    <bias_mean>0.1</bias_mean>
+                    <bias_stddev>0.001</bias_stddev>
+                </noise>
+                </y>
+                <z>
+                <noise type="gaussian">
+                    <mean>0.0</mean>
+                    <stddev>1.7e-2</stddev>
+                    <bias_mean>0.1</bias_mean>
+                    <bias_stddev>0.001</bias_stddev>
+                </noise>
+                </z>
+            </linear_acceleration>
+            </imu>
+        </sensor>
+    </gazebo>
     <gazebo reference="camera_link">
         <sensor type="depth" name="guard_cam">

File: greenguard_description/urdf/my_robot.urdf (robot description, URDF)
Before this commit: robot greenguard, 8 links, 7 joints
Links:
- removed link dummy_link
Joints:
- removed joint dummy_joint
